File: attachmentBoard.kicad_sch (KiCad schematic)
At the start: 33 parts, among them IC1 L7805CD2T-TR, J1 B4B-XH-A, J11 Conn_01x03, J12 Conn_01x03, J13 Conn_01x03, J14 Conn_01x03, J15 Conn_01x03, J16 Conn_01x03, J17 Conn_01x03, J18 Conn_01x03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

Commit message: Changed capacitor values on 12v convertor
Parts:
- C2: value .33uF -> 1uF
- C3: value 1uF -> .22uF
Changed lines of the file:
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@@
       (effects (font (size 1.27 1.27)) (justify left))
     )
-    (property "Value" "1uF" (at 73.66 167.005 0)
+    (property "Value" ".22uF" (at 73.66 167.005 0)
       (effects (font (size 1.27 1.27)) (justify left))
     )
@@
       (effects (font (size 1.27 1.27)) (justify left))
     )
-    (property "Value" ".33uF" (at 41.91 168.275 0)
-      (effects (font (size 1.27 1.27)) (justify left))
-    )
+    (property "Value" "1uF" (at 41.91 168.275 0)
+      (effects (font (size 1.27 1.27)) (justify left))
+    )
